Commit message: Imported upstream version '0.3.6' of 'upstream'

File: motoman_sia10d_support/urdf/sia10d.urdf (robot description, URDF)
Before this commit: robot motoman_sia10d, 9 links, 8 joints
Links:
- added link base
Joints:
- added joint link_l-base: type fixed, parent link_l, child base, origin xyz=0 0 0 rpy=0 0 0
- joint joint_b: limit lower=-1.91 upper=1.91 effort=100 velocity=3.48 -> lower=-1.9198 upper=1.9198 effort=100 velocity=3.4906
- joint joint_e: limit lower=-2.96 upper=2.96 effort=100 velocity=2.96 -> lower=-2.9670 upper=2.9670 effort=100 velocity=2.9670
- joint joint_l: limit lower=-1.91 upper=1.91 effort=100 velocity=2.96 -> lower=-1.9198 upper=1.9198 effort=100 velocity=2.9670
- joint joint_r: limit lower=-3.1416 upper=3.1416 effort=100 velocity=3.48 -> lower=-3.1415 upper=3.1415 effort=100 velocity=3.4906
- joint joint_s: limit lower=-3.1416 upper=3.1416 effort=100 velocity=2.96 -> lower=-3.1415 upper=3.1415 effort=100 velocity=2.9670
- joint joint_t: limit lower=-3.1416 upper=3.1416 effort=100 velocity=6.97 -> lower=-3.1415 upper=3.1415 effort=100 velocity=6.9813
- joint joint_u: limit lower=-2.35 upper=2.35 effort=100 velocity=2.96 -> lower=-2.3561 upper=2.3561 effort=100 velocity=2.9670

File: motoman_sia10d_support/urdf/sia10d_macro.xacro (robot description, xacro)
@@ -225,5 +225,5 @@
 			<origin xyz="0 0 0.36" rpy="0 0 0"/>
 			<axis xyz="0 0 1" />
-			<limit lower="-3.1416" upper="3.1416" effort="100" velocity="2.96" />
+			<limit lower="-3.1415" upper="3.1415" effort="100" velocity="2.9670" />
 		</joint>
 		<joint name="${prefix}joint_l" type="revolute">
@@ -232,5 +232,5 @@
 			<origin xyz="0 0 0" rpy="0 0 0"/>
 			<axis xyz="0 1 0" />
-			<limit lower="-1.91" upper="1.91" effort="100" velocity="2.96" />
+			<limit lower="-1.9198" upper="1.9198" effort="100" velocity="2.9670" />
 		</joint>
 		<joint name="${prefix}joint_e" type="revolute">
@@ -239,5 +239,5 @@
 			<origin xyz="0 0 0.36" rpy="0 0 0"/>
 			<axis xyz="0 0 1" />
-			<limit lower="-2.96" upper="2.96" effort="100" velocity="2.96" />
+			<limit lower="-2.9670" upper="2.9670" effort="100" velocity="2.9670" />
 		</joint>
 		<joint name="${prefix}joint_u" type="revolute">
@@ -246,5 +246,5 @@
 			<origin xyz="0 0 0" rpy="0 0 0"/>
 			<axis xyz="0 -1 0" />
-			<limit lower="-2.35" upper="2.35" effort="100" velocity="2.96" />
+			<limit lower="-2.3561" upper="2.3561" effort="100" velocity="2.9670" />
 		</joint>
 		<joint name="${prefix}joint_r" type="revolute">
@@ -253,5 +253,5 @@
 			<origin xyz="0 0 0.360" rpy="0 0 0"/>
 			<axis xyz="0 0 -1" />
-			<limit lower="-3.1416" upper="3.1416" effort="100" velocity="3.48" />
+			<limit lower="-3.1415" upper="3.1415" effort="100" velocity="3.4906" />
 		</joint>
 		<joint name="${prefix}joint_b" type="revolute">
@@ -260,5 +260,5 @@
 			<origin xyz="0 0 0" rpy="0 0 0"/>
 			<axis xyz="0 -1 0" />
-			<limit lower="-1.91" upper="1.91" effort="100" velocity="3.48" />
+			<limit lower="-1.9198" upper="1.9198" effort="100" velocity="3.4906" />
 		</joint>
 		<joint name="${prefix}joint_t" type="revolute">
@@ -267,7 +267,14 @@
 			<origin xyz="0 0 0.155" rpy="0 0 0"/>
 			<axis xyz="0 0 -1" />
-			<limit lower="-3.1416" upper="3.1416" effort="100" velocity="6.97" />
+			<limit lower="-3.1415" upper="3.1415" effort="100" velocity="6.9813" />
 		</joint>
 		<!-- end of joint list -->
+		<!-- ROS base_link (via link_l) to Motoman Robot (not Base) Frame transform -->
+		<link name="${prefix}base" />
+		<joint name="${prefix}link_l-base" type="fixed">
+			<origin xyz="0 0 0" rpy="0 0 0"/>
+			<parent link="${prefix}link_l"/>
+			<child link="${prefix}base"/>
+		</joint>
 	</xacro:macro>
 </robot>

File: motoman_sia10f_support/urdf/sia10f.urdf (robot description, URDF)
Before this commit: robot motoman_sia10f, 8 links, 7 joints
Links:
- added link base
Joints:
- added joint link_l-base: type fixed, parent link_l, child base, origin xyz=0 0 0 rpy=0 0 0
- joint joint_b: limit lower=-1.91 upper=1.91 effort=100 velocity=3.48 -> lower=-1.9198 upper=1.9198 effort=100 velocity=3.4906
- joint joint_e: limit lower=-2.96 upper=2.96 effort=100 velocity=2.96 -> lower=-2.9670 upper=2.9670 effort=100 velocity=2.9670
- joint joint_l: limit lower=-1.91 upper=1.91 effort=100 velocity=2.96 -> lower=-1.9198 upper=1.9198 effort=100 velocity=2.9670
- joint joint_r: limit lower=-3.1416 upper=3.1416 effort=100 velocity=3.48 -> lower=-3.1415 upper=3.1415 effort=100 velocity=3.4906
- joint joint_s: limit lower=-3.1416 upper=3.1416 effort=100 velocity=2.96 -> lower=-3.1415 upper=3.1415 effort=100 velocity=2.9670
- joint joint_t: limit lower=-3.1416 upper=3.1416 effort=100 velocity=6.97 -> lower=-3.1415 upper=3.1415 effort=100 velocity=6.9813
- joint joint_u: limit lower=-2.35 upper=2.35 effort=100 velocity=2.96 -> lower=-2.3561 upper=2.3561 effort=100 velocity=2.9670

File: motoman_sia10f_support/urdf/sia10f_macro.xacro (robot description, xacro)
@@ -139,5 +139,5 @@
 			<origin xyz="0 0 0.36" rpy="0 0 0"/>
 			<axis xyz="0 0 1" />
-			<limit lower="-3.1416" upper="3.1416" effort="0" velocity="2.96" />
+			<limit lower="-3.1415" upper="3.1415" effort="0" velocity="2.9670" />
 		</joint>
 		<joint name="${prefix}joint_2_l" type="revolute">
@@ -146,5 +146,5 @@
 			<origin xyz="0 0 0" rpy="0 0 0"/>
 			<axis xyz="0 1 0" />
-			<limit lower="-1.91" upper="1.91" effort="0" velocity="2.96" />
+			<limit lower="-1.9198" upper="1.9198" effort="0" velocity="2.9670" />
 		</joint>
 		<joint name="${prefix}joint_3_e" type="revolute">
@@ -153,5 +153,5 @@
 			<origin xyz="0 0 0.36" rpy="0 0 0"/>
 			<axis xyz="0 0 1" />
-			<limit lower="-2.96" upper="2.96" effort="0" velocity="2.96" />
+			<limit lower="-2.9670" upper="2.9670" effort="0" velocity="2.9670" />
 		</joint>
 		<joint name="${prefix}joint_4_u" type="revolute">
@@ -160,5 +160,5 @@
 			<origin xyz="0 0 0" rpy="0 0 0"/>
 			<axis xyz="0 -1 0" />
-			<limit lower="-2.35" upper="2.35" effort="0" velocity="2.96" />
+			<limit lower="-2.3561" upper="2.3561" effort="0" velocity="2.9670" />
 		</joint>
 		<joint name="${prefix}joint_5_r" type="revolute">
@@ -167,5 +167,5 @@
 			<origin xyz="0 0 0.360" rpy="0 0 0"/>
 			<axis xyz="0 0 -1" />
-			<limit lower="-3.1416" upper="3.1416" effort="0" velocity="3.48" />
+			<limit lower="-3.1415" upper="3.1415" effort="0" velocity="3.4906" />
 		</joint>
 		<joint name="${prefix}joint_6_b" type="revolute">
@@ -174,5 +174,5 @@
 			<origin xyz="0 0 0" rpy="0 0 0"/>
 			<axis xyz="0 -1 0" />
-			<limit lower="-1.91" upper="1.91" effort="0" velocity="3.48" />
+			<limit lower="-1.9198" upper="1.9198" effort="0" velocity="3.4906" />
 		</joint>
 		<joint name="${prefix}joint_7_t" type="revolute">
@@ -181,12 +181,19 @@
 			<origin xyz="0 0 0.155" rpy="0 0 0"/>
 			<axis xyz="0 0 -1" />
-			<limit lower="-3.1416" upper="3.1416" effort="0" velocity="6.97" />
+			<limit lower="-3.1415" upper="3.1415" effort="0" velocity="6.9813" />
 		</joint>
     <joint name="${prefix}joint_tool0" type="fixed" >
-      <origin xyz="0 0 0.0" rpy="0 0 -3.1416"/>
+      <origin xyz="0 0 0.0" rpy="0 0 -3.1415926535"/>
       <parent link="${prefix}link_7_t" />
       <child link="${prefix}link_tool0" />
     </joint>
 		<!-- end of joint list -->
+		<!-- ROS base_link (via link_l) to Motoman Robot (not Base) Frame transform -->
+		<link name="${prefix}base" />
+		<joint name="${prefix}link_2_l-base" type="fixed">
+			<origin xyz="0 0 0" rpy="0 0 0"/>
+			<parent link="${prefix}link_2_l"/>
+			<child link="${prefix}base"/>
+		</joint>
 	</xacro:macro>
 </robot>

File: motoman_sia20d_support/urdf/sia20d.urdf (robot description, URDF)
Before this commit: robot motoman_sia20d, 9 links, 8 joints
Links:
- added link base
Joints:
- added joint link_l-base: type fixed, parent link_l, child base, origin xyz=0 0 0 rpy=0 0 0
- joint joint_b: limit lower=-1.91 upper=1.91 effort=100 velocity=3.48 -> lower=-1.9198 upper=1.9198 effort=100 velocity=3.4906
- joint joint_e: limit lower=-2.96 upper=2.96 effort=100 velocity=2.96 -> lower=-2.9670 upper=2.9670 effort=100 velocity=2.9670
- joint joint_l: limit lower=-1.91 upper=1.91 effort=100 velocity=2.26 -> lower=-1.9198 upper=1.9198 effort=100 velocity=2.2689
- joint joint_r: limit lower=-3.1416 upper=3.1416 effort=100 velocity=3.48 -> lower=-3.1415 upper=3.1415 effort=100 velocity=3.4906
- joint joint_s: limit lower=-3.1416 upper=3.1416 effort=100 velocity=2.26 -> lower=-3.1415 upper=3.1415 effort=100 velocity=2.2689
- joint joint_t: limit lower=-3.1416 upper=3.1416 effort=100 velocity=6.97 -> lower=-3.1415 upper=3.1415 effort=100 velocity=6.9813
- joint joint_u: limit lower=-2.26 upper=2.26 effort=100 velocity=2.96 -> lower=-2.2689 upper=2.2689 effort=100 velocity=2.9670

File: motoman_sia20d_support/urdf/sia20d_macro.xacro (robot description, xacro)
@@ -141,5 +141,5 @@
 			<origin xyz="0 0 0.41" rpy="0 0 0"/>
 			<axis xyz="0 0 1" />
-			<limit lower="-3.1416" upper="3.1416" effort="100" velocity="2.26" />
+			<limit lower="-3.1415" upper="3.1415" effort="100" velocity="2.2689" />
 		</joint>
 		<joint name="${prefix}joint_l" type="revolute">
@@ -148,5 +148,5 @@
 			<origin xyz="0 0 0" rpy="0 0 0"/>
 			<axis xyz="0 1 0" />
-			<limit lower="-1.91" upper="1.91" effort="100" velocity="2.26" />
+			<limit lower="-1.9198" upper="1.9198" effort="100" velocity="2.2689" />
 		</joint>
 		<joint name="${prefix}joint_e" type="revolute">
@@ -155,5 +155,5 @@
 			<origin xyz="0 0 0.49" rpy="0 0 0"/>
 			<axis xyz="0 0 1" />
-			<limit lower="-2.96" upper="2.96" effort="100" velocity="2.96" />
+			<limit lower="-2.9670" upper="2.9670" effort="100" velocity="2.9670" />
 		</joint>
 		<joint name="${prefix}joint_u" type="revolute">
@@ -162,5 +162,5 @@
 			<origin xyz="0 0 0" rpy="0 0 0"/>
 			<axis xyz="0 -1 0" />
-			<limit lower="-2.26" upper="2.26" effort="100" velocity="2.96" />
+			<limit lower="-2.2689" upper="2.2689" effort="100" velocity="2.9670" />
 		</joint>
 		<joint name="${prefix}joint_r" type="revolute">
@@ -169,5 +169,5 @@
 			<origin xyz="0 0 0.420" rpy="0 0 0"/>
 			<axis xyz="0 0 -1" />
-			<limit lower="-3.1416" upper="3.1416" effort="100" velocity="3.48" />
+			<limit lower="-3.1415" upper="3.1415" effort="100" velocity="3.4906" />
 		</joint>
 		<joint name="${prefix}joint_b" type="revolute">
@@ -176,5 +176,5 @@
 			<origin xyz="0 0 0" rpy="0 0 0"/>
 			<axis xyz="0 -1 0" />
-			<limit lower="-1.91" upper="1.91" effort="100" velocity="3.48" />
+			<limit lower="-1.9198" upper="1.9198" effort="100" velocity="3.4906" />
 		</joint>
 		<joint name="${prefix}joint_t" type="revolute">
@@ -183,12 +183,19 @@
 			<origin xyz="0 0 0.18" rpy="0 0 0"/>
 			<axis xyz="0 0 -1" />
-			<limit lower="-3.1416" upper="3.1416" effort="100" velocity="6.97" />
+			<limit lower="-3.1415" upper="3.1415" effort="100" velocity="6.9813" />
 		</joint>
     <joint name="${prefix}link_t-tool0" type="fixed" >
-      <origin xyz="0 0 0.0" rpy="0 0 -3.1416"/>
+      <origin xyz="0 0 0.0" rpy="0 0 -3.1415926535"/>
       <parent link="${prefix}link_t" />
       <child link="${prefix}tool0" />
     </joint>
 		<!-- end of joint list -->
+		<!-- ROS base_link (via link_l) to Motoman Robot (not Base) Frame transform -->
+		<link name="${prefix}base" />
+		<joint name="${prefix}link_l-base" type="fixed">
+			<origin xyz="0 0 0" rpy="0 0 0"/>
+			<parent link="${prefix}link_l"/>
+			<child link="${prefix}base"/>
+		</joint>
 	</xacro:macro>
 </robot>

File: motoman_sia5d_support/urdf/sia5d.urdf (robot description, URDF)
Before this commit: robot motoman_sia5d, 9 links, 8 joints
Links:
- added link base
Joints:
- added joint link_l-base: type fixed, parent link_l, child base, origin xyz=0 0 0 rpy=0 0 0

File: motoman_sia5d_support/urdf/sia5d_macro.xacro (robot description, xacro)
@@ -171,4 +171,11 @@
     <child link="${prefix}tool0" />
   </joint>
+    <!-- ROS base_link (via link_l) to Motoman Robot (not Base) Frame transform -->
+    <link name="${prefix}base" />
+    <joint name="${prefix}link_l-base" type="fixed">
+      <origin xyz="0 0 0" rpy="0 0 0"/>
+      <parent link="${prefix}link_l"/>
+      <child link="${prefix}base"/>
+    </joint>
 	</xacro:macro>
 </robot>
